Commit message: update urdf, ik node, add new meshes

File: urdf/my_arm.urdf (robot description, URDF)
Before this commit: robot my_arm, 9 links, 8 joints
Links:
- added link gripper_base; visual mesh filename=package://my_arm_description/meshes/visual/gripper_base.stl
- added link joint_without_idler2; visual mesh filename=package://my_arm_description/meshes/visual/joint_without_id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
Joints:
- added joint gripperlink_to_joint_without_idler2: type fixed, parent gripper_link2, child joint_without_idler2, origin xyz=-0.017 -0.0352 -0.0115 rpy=1.5708 -1.5708 0
- added joint joint_without_idler2_to_gripper_base: type fixed, parent joint_without_idler2, child gripper_base, origin xyz=0.002 -0.0119 0.007 rpy=-3.1416 0 0
